File: DC-STB-X8.brd (EAGLE design)
At the start: 29 x 87 mm, 4 parts

Commit message: Added logos to all boards. Generated CAM files.
Parts:
- added LOGO1: MFDECLOGO_L_10MM, _my_logos:MFDEC_L_10MM
- added LOGO2: RSNURL_QR_10MM, _my_logos:RSNURL_QR_10MM
Changed lines of the file:
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@@
 <drawing>
 <settings>
-<setting alwaysvectorfont="no"/>
+<setting alwaysvectorfont="yes"/>
 <setting verticaltext="up"/>
 </settings>
@@
 <layer number="97" name="Info" color="7" fill="1" visible="no" active="no"/>
 <layer number="98" name="Guide" color="6" fill="1" visible="no" active="no"/>
+<layer number="200" name="200bmp" color="1" fill="10" visible="yes" active="yes"/>
 </layers>
 <board>
@@
 <element name="U$3" library="KF8500-Terminals" package="KF8500-8.5-2P" value="KF8500-8.5-2P" x="15" y="52" smashed="yes" rot="R90"/>
 <element name="U$4" library="KF8500-Terminals" package="KF8500-8.5-2P" value="KF8500-8.5-2P" x="15" y="69" smashed="yes" rot="R90"/>
+<element name="LOGO1" library="_my_logos" package="MFDEC_L_10MM" value="MFDECLOGO_L_10MM" x="15" y="75" smashed="yes" rot="MR0"/>
+<element name="LOGO2" library="_my_logos" package="RSNURL_QR_10MM" value="RSNURL_QR_10MM" x="10" y="1" smashed="yes" rot="MR0"/>
 </elements>
 <signals>
